File: Week 1.kicad_sch (KiCad schematic)
At the start: 7 parts, among them J1 Conn_01x04_Pin, J2 Conn_01x08_Pin, SW1 SW_Push, SW2 SW_Push, U1 XIAO-ESP32-C3-SMD, U2 DHT11

Commit message: added many things
Connections:
- net DHT11 DATA: now also U1.2 (D1)
- net GPIO 2: now also U1.3 (D2)
- net GPIO 3: now also U1.4 (D3)
- net SCL: now also J1.3 (Pin_3), J2.3 (Pin_3), U1.5 (D4)
- net SDA: now also J1.4 (Pin_4), J2.4 (Pin_4), U1.6 (D5)
Other:
- note removed: "SCL"
Changed lines of the file:
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@@
-		)
-	)
-	(text "SCL"
-		(exclude_from_sim no)
-		(at 218.44 120.142 90)
-		(effects
-			(font
-				(size 1.27 1.27)
-			)
 		)
 	)
@@
 	(wire
 		(pts
-			(xy 224.79 163.83) (xy 226.06 163.83)
-		)
-		(stroke
-			(width 0)
-			(type default)
-		)
-	)
-	(wire
-		(pts
 			(xy 220.98 146.05) (xy 226.06 146.05)
 		)
@@
 	(wire
 		(pts
+			(xy 210.82 54.61) (xy 217.17 54.61)
+		)
+		(stroke
+			(width 0)
+			(type default)
+		)
+	)
+	(wire
+		(pts
 			(xy 250.19 120.65) (xy 256.54 120.65)
 		)
@@
 	(wire
 		(pts
+			(xy 210.82 66.04) (xy 217.17 66.04)
+		)
+		(stroke
+			(width 0)
+			(type default)
+		)
+	)
+	(wire
+		(pts
 			(xy 236.22 22.86) (xy 240.03 22.86)
 		)
@@
 	(wire
 		(pts
+			(xy 210.82 50.8) (xy 217.17 50.8)
+		)
+		(stroke
+			(width 0)
+			(type default)
+		)
+	)
+	(wire
+		(pts
 			(xy 220.98 111.76) (xy 220.98 121.92)
 		)
@@
 	(wire
 		(pts
+			(xy 210.82 58.42) (xy 217.17 58.42)
+		)
+		(stroke
+			(width 0)
+			(type default)
+		)
+	)
+	(wire
+		(pts
 			(xy 213.36 153.67) (xy 213.36 156.21)
 		)
@@
 	(wire
 		(pts
+			(xy 210.82 62.23) (xy 217.17 62.23)
+		)
+		(stroke
+			(width 0)
+			(type default)
+		)
+	)
+	(wire
+		(pts
 			(xy 223.52 111.76) (xy 223.52 114.3)
 		)
@@
 	)
 	(label "SDA"
-		(at 217.17 121.92 90)
+		(at 215.9 118.11 90)
 		(effects
 			(font
@@
 		)
 	)
+	(label "SCL"
+		(at 218.44 118.11 90)
+		(effects
+			(font
+				(size 1.27 1.27)
+			)
+			(justify left bottom)
+		)
+	)
 	(label "DHT11 DATA"
 		(at 226.06 146.05 0)
@@
 		)
 	)
+	(label "GPIO 2"
+		(at 210.82 54.61 0)
+		(effects
+			(font
+				(size 1.27 1.27)
+			)
+			(justify left bottom)
+		)
+	)
 	(label "GPIO 3"
 		(at 250.19 120.65 0)
@@
 		)
 	)
+	(label "SCL"
+		(at 210.82 62.23 0)
+		(effects
+			(font
+				(size 1.27 1.27)
+			)
+			(justify left bottom)
+		)
+	)
 	(label "ESP32 C3"
 		(at 269.24 19.05 0)
@@
 	)
 	(label "DHT11 DATA"
-		(at 226.06 163.83 0)
+		(at 210.82 50.8 0)
+		(effects
+			(font
+				(size 1.27 1.27)
+			)
+			(justify left bottom)
+		)
+	)
+	(label "DHT11 DATA"
+		(at 224.79 163.83 0)
 		(effects
 			(font
@@
 	)
 	(label "SDA"
-		(at 265.43 151.13 0)
+		(at 265.43 149.86 0)
+		(effects
+			(font
+				(size 1.27 1.27)
+			)
+			(justify left bottom)
+		)
+	)
+	(label "SDA"
+		(at 210.82 66.04 0)
 		(effects
 			(font
@@
 	)
 	(label "SCL"
-		(at 265.43 148.59 0)
-		(effects
-			(font
+		(at 265.43 147.32 0)
+		(effects
+			(font
+				(size 1.27 1.27)
+			)
+			(justify left bottom)
+		)
+	)
+	(label "GPIO 3"
+		(at 210.82 58.42 0)
+		(effects
+			(font
